File: KiCAD/RAM_ROM_Interface.kicad_sch (KiCad schematic)
At the start: 2 parts

Commit message: Update to V9
Connections:
- net ~{MEM}: no longer Z67.5, Z68.5
- new net D2: Z68.5
- new net D6: Z67.5
Changed lines of the file:
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@@
 (kicad_sch
-	(version 20231120)
+	(version 20250114)
 	(generator "eeschema")
-	(generator_version "8.0")
+	(generator_version "9.0")
 	(paper "USLetter")
 	(title_block
@@
 	)
 	(junction
-		(at 224.79 100.33)
-		(diameter 0)
-		(color 0 0 0 0)
-	)
-	(junction
 		(at 83.185 68.58)
 		(diameter 0)
 		(color 0 0 0 0)
 	)
-	(junction
-		(at 138.43 74.93)
-		(diameter 0)
-		(color 0 0 0 0)
-	)
 	(bus_entry
 		(at 31.75 97.79)
@@
 	(wire
 		(pts
-			(xy 224.79 100.33) (xy 262.89 100.33)
+			(xy 210.82 100.33) (xy 262.89 100.33)
 		)
 		(stroke
@@
 	(wire
 		(pts
-			(xy 138.43 74.93) (xy 262.89 74.93)
+			(xy 124.46 74.93) (xy 262.89 74.93)
 		)
 		(stroke
@@
 	(wire
 		(pts
-			(xy 210.82 100.33) (xy 224.79 100.33)
-		)
-		(stroke
-			(width 0)
-			(type default)
-		)
-	)
-	(wire
-		(pts
 			(xy 167.64 87.63) (xy 262.89 87.63)
 		)
@@
 		(pts
 			(xy 102.87 68.58) (xy 262.89 68.58)
-		)
-		(stroke
-			(width 0)
-			(type default)
-		)
-	)
-	(wire
-		(pts
-			(xy 124.46 74.93) (xy 138.43 74.93)
 		)
 		(stroke
@@
 	(label "D0"
 		(at 262.255 113.03 180)
-		(fields_autoplaced yes)
 		(effects
 			(font
@@
 	(label "ROMD4"
 		(at 34.29 87.63 0)
-		(fields_autoplaced yes)
 		(effects
 			(font
@@
 	(label "ROMD0"
 		(at 34.29 113.03 0)
-		(fields_autoplaced yes)
 		(effects
 			(font
@@
 	(label "D2"
 		(at 262.255 100.33 180)
-		(fields_autoplaced yes)
 		(effects
 			(font
@@
 	(label "RAMD4"
 		(at 147.955 124.46 270)
-		(fields_autoplaced yes)
 		(effects
 			(font
@@
 	(label "D7"
 		(at 262.255 68.58 180)
-		(fields_autoplaced yes)
 		(effects
 			(font
@@
 	(label "RAMD3"
 		(at 169.545 124.46 270)
-		(fields_autoplaced yes)
 		(effects
 			(font
@@
 	(label "D3"
 		(at 262.255 93.98 180)
-		(fields_autoplaced yes)
 		(effects
 			(font
@@
 	(label "ROMD6"
 		(at 34.29 74.93 0)
-		(fields_autoplaced yes)
 		(effects
 			(font
@@
 	(label "RAMD2"
 		(at 191.135 124.46 270)
-		(fields_autoplaced yes)
 		(effects
 			(font
@@
 	(label "ROMD7"
 		(at 34.29 68.58 0)
-		(fields_autoplaced yes)
 		(effects
 			(font
@@
 	(label "RAMD0"
 		(at 234.315 124.46 270)
-		(fields_autoplaced yes)
 		(effects
 			(font
@@
 	(label "RAMD1"
 		(at 212.725 124.46 270)
-		(fields_autoplaced yes)
 		(effects
 			(font
@@
 	(label "D6"
 		(at 262.255 74.93 180)
-		(fields_autoplaced yes)
 		(effects
 			(font
@@
 	(label "D1"
 		(at 262.255 106.68 180)
-		(fields_autoplaced yes)
 		(effects
 			(font
@@
 	(label "ROMD2"
 		(at 34.29 100.33 0)
-		(fields_autoplaced yes)
 		(effects
 			(font
@@
 	(label "D4"
 		(at 262.255 87.63 180)
-		(fields_autoplaced yes)
 		(effects
 			(font
@@
 	(label "ROMD5"
 		(at 34.29 81.28 0)
-		(fields_autoplaced yes)
 		(effects
 			(font
@@
 	(label "ROMD1"
 		(at 34.29 106.68 0)
-		(fields_autoplaced yes)
 		(effects
 			(font
@@
 	(label "RAMD6"
 		(at 104.775 124.46 270)
-		(fields_autoplaced yes)
 		(effects
 			(font
@@
 	(label "RAMD5"
 		(at 126.365 124.46 270)
-		(fields_autoplaced yes)
 		(effects
 			(font
@@
 	(label "ROMD3"
 		(at 34.29 93.98 0)
-		(fields_autoplaced yes)
 		(effects
 			(font
@@
 	(label "RAMD7"
 		(at 83.185 124.46 270)
-		(fields_autoplaced yes)
 		(effects
 			(font
@@
 	(label "D5"
 		(at 262.255 81.28 180)
-		(fields_autoplaced yes)
 		(effects
 			(font
@@
 		(shape bidirectional)
 		(at 265.43 63.5 90)
-		(fields_autoplaced yes)
 		(effects
 			(font
@@
 		(shape bidirectional)
 		(at 27.94 134.62 180)
-		(fields_autoplaced yes)
 		(effects
 			(font
@@
 		(shape bidirectional)
 		(at 27.94 66.04 180)
-		(fields_autoplaced yes)
 		(effects
 			(font
@@
 		(shape input)
 		(at 27.94 42.545 180)
-		(fields_autoplaced yes)
-		(effects
-			(font
+		(effects
+			(font
